Commit message: Gazebo simulation working with diff_drive

File: src/mek_lilrobot/description/robot_core.xacro (robot description, xacro)
@@ -1,4 +1,5 @@
 <?xml version="1.0"?>
 <robot xmlns:xacro="http://www.ros.org/wiki/xacro">
+    <xacro:include filename="inertial_macros.xacro"/>
     <material name="white">
         <color rgba="1 1 1 1" />
@@ -21,11 +22,16 @@
             <material name="white" />
         </visual>
+        <collision>
+            <geometry>
+                <box size="0.1222 0.10825 0.005" />
+            </geometry>
+        </collision>
+        <xacro:inertial_box mass="0.5" x="0.1222" y="0.10825" z="0.005">
+            <origin xyz="0 0 0" rpy="0 0 0" />
+        </xacro:inertial_box>
     </link>
-    <!--<joint name="right_wheel_joint" type="continuous">
-        <parent link="base_link" />
-        <child link="right_wheel" />
-        <origin xyz="0 -0.0675 0.02175" rpy="1.57079632679 0 0"/>
-        <axis xyz="0 0 -1"/>
-    </joint>-->
+    <gazebo reference="chassis">
+        <material>Gazebo/White</material>
+    </gazebo>
     <joint name="right_wheel_joint" type="continuous">
         <parent link="base_link" />
@@ -41,5 +47,16 @@
             <material name="black"/>
         </visual>
+        <collision>
+            <geometry>
+                <cylinder radius="0.02175" length="0.009"/>
+            </geometry>
+        </collision>
+        <xacro:inertial_cylinder mass="0.05" radius="0.02175" length="0.009">
+            <origin xyz="0 0 0" rpy="0 0 0"/>
+        </xacro:inertial_cylinder>
     </link>
+    <gazebo reference="right_wheel">
+        <material>Gazebo/Black</material>
+    </gazebo>
     <joint name="left_wheel_joint" type="continuous">
         <parent link="base_link" />
@@ -55,5 +72,16 @@
             <material name="black"/>
         </visual>
+        <collision>
+            <geometry>
+                <cylinder radius="0.02175" length="0.009"/>
+            </geometry>
+        </collision>
+        <xacro:inertial_cylinder mass="0.05" radius="0.02175" length="0.009">
+            <origin xyz="0 0 0" rpy="0 0 0"/>
+        </xacro:inertial_cylinder>
     </link>
+    <gazebo reference="left_wheel">
+        <material>Gazebo/Black</material>
+    </gazebo>
     <joint name="caster_wheel_joint" type="fixed">
         <parent link="base_link"/>
@@ -68,4 +96,17 @@
             <material name="black"/>
         </visual>
+        <collision>
+            <geometry>
+                <sphere radius="0.008"/>
+            </geometry>
+        </collision>
+        <xacro:inertial_sphere mass="0.01" radius="0.008">
+            <origin xyz="0 0 0" rpy="0 0 0"/>
+        </xacro:inertial_sphere>
     </link>
+    <gazebo reference="caster_wheel">
+        <material>Gazebo/Black</material>
+        <mu1 value="0.001"/>
+        <mu2 value="0.001"/>
+    </gazebo>
 </robot>

Commit message: Add camera to simulation

File: src/mek_lilrobot/description/robot_core.xacro (robot description, xacro)
@@ -7,4 +7,7 @@
     <material name="black">
         <color rgba="0 0 0 1" />
+    </material>
+    <material name="red">
+        <color rgba="1 0 0 1"/>
     </material>
     <link name="base_link">
@@ -110,3 +113,45 @@
         <mu2 value="0.001"/>
     </gazebo>
+    <joint name="camera_joint" type="fixed">
+        <parent link="base_link"/>
+        <child link="camera_link"/>
+        <origin xyz="-0.062 0 0.119" rpy="0 0.26 0"/>
+    </joint>
+    <link name="camera_link">
+        <visual>
+            <geometry>
+                <box size="0.010 0.03 0.03"/>
+            </geometry>
+            <material name="red"/>
+        </visual>
+    </link>
+    <gazebo reference="camera_link">
+        <material>Gazebo/Red</material>
+        <sensor name="camera" type="camera">
+            <pose> 0 0 0 0 0 0 </pose>
+            <visualize>true</visualize>
+            <update_rate>10</update_rate>
+            <camera>
+                <horizontal_fov>0.942</horizontal_fov>
+                <image>
+                    <format>R8G8B8</format>
+                    <width>640</width>
+                    <height>480</height>
+                </image>
+                <clip>
+                    <near>0.05</near>
+                    <far>8.0</far>
+                </clip>
+            </camera>
+            <plugin name="camera_controller" filename="libgazebo_ros_camera.so">
+                <frame_name>camera_link_optical</frame_name>
+            </plugin>
+        </sensor>
+    </gazebo>
+    <joint name="camera_optical_joint" type="fixed">
+        <origin xyz="0 0 0" rpy="${-pi/2} 0 ${-pi/2}" />
+        <parent link="camera_link" />
+        <child link="camera_link_optical" />
+    </joint>
+    <link name="camera_link_optical"></link>
 </robot>

Commit message: Add laser range sensor to URDF

File: src/mek_lilrobot/description/robot_core.xacro (robot description, xacro)
@@ -155,3 +155,54 @@
     </joint>
     <link name="camera_link_optical"></link>
+    <joint name="laser_joint" type="fixed">
+        <parent link="base_link"/>
+        <child link="laser_link"/>
+        <origin xyz="0.011 0.00 0.01675" rpy="0 0 0"/>
+    </joint>
+    <link name="laser_link">
+        <visual>
+            <geometry>
+                <box size="0.002 0.005 0.005"/>
+            </geometry>
+            <material name="red"/>
+        </visual>
+    </link>
+    <gazebo reference="laser_link">
+        <material>Gazebo/Red</material>
+        <selfCollide>0</selfCollide>
+        <sensor type="ray" name="laser_link">
+            <pose>0.0025 0 0 0 0 0</pose>
+            <visualize>true</visualize>
+            <update_rate>10</update_rate>
+            <ray>
+                <scan>
+                    <horizontal>
+                        <samples>10</samples>
+                        <resolution>1</resolution>
+                        <min_angle>-0.174533</min_angle>
+                        <max_angle>0.174533</max_angle>
+                    </horizontal>
+                    <vertical>
+                        <samples>10</samples>
+                        <resolution>1</resolution>
+                        <min_angle>-0.174533</min_angle>
+                        <max_angle>0.174533</max_angle>
+                    </vertical>
+                </scan>
+                <range>
+                    <min>0.001</min>
+                    <max>0.5</max>
+                    <resolution>0.001</resolution>
+                </range>
+            </ray>
+            <update_rate>10</update_rate>
+            <plugin name="gazebo_ros_range_controller" filename="libgazebo_ros_ray_sensor.so">
+                <ros>
+                    <remapping>~/out:=laser</remapping>
+                </ros>
+                <output_type>sensor_msgs/Range</output_type>
+                <!-- <frame_name> ommited, will default to range_link -->
+            </plugin>
+        </sensor>
+    </gazebo>
 </robot>

Commit message: Fix robot drifting in simulation

File: src/mek_lilrobot/description/robot_core.xacro (robot description, xacro)
@@ -52,8 +52,16 @@
         <collision>
             <geometry>
-                <cylinder radius="0.02175" length="0.009"/>
-            </geometry>
-        </collision>
-        <xacro:inertial_cylinder mass="0.05" radius="0.02175" length="0.009">
+                <sphere radius="0.02175"/>
+            </geometry>
+            <surface>
+                <contact>
+                    <ode>
+                        <kp>1e15</kp>
+                        <kd>1e13</kd>
+                    </ode>
+                </contact>
+            </surface>
+        </collision>
+        <xacro:inertial_cylinder mass="0.5" radius="0.02175" length="0.009">
             <origin xyz="0 0 0" rpy="0 0 0"/>
         </xacro:inertial_cylinder>
@@ -61,4 +69,6 @@
     <gazebo reference="right_wheel">
         <material>Gazebo/Black</material>
+        <mu1 value="0.8"/>
+        <mu2 value="0.8"/>
     </gazebo>
     <joint name="left_wheel_joint" type="continuous">
@@ -77,8 +87,16 @@
         <collision>
             <geometry>
-                <cylinder radius="0.02175" length="0.009"/>
-            </geometry>
-        </collision>
-        <xacro:inertial_cylinder mass="0.05" radius="0.02175" length="0.009">
+                <sphere radius="0.02175"/>
+            </geometry>
+            <surface>
+                <contact>
+                    <ode>
+                        <kp>1e15</kp>
+                        <kd>1e13</kd>
+                    </ode>
+                </contact>
+            </surface>
+        </collision>
+        <xacro:inertial_cylinder mass="0.5" radius="0.02175" length="0.009">
             <origin xyz="0 0 0" rpy="0 0 0"/>
         </xacro:inertial_cylinder>
@@ -86,4 +104,6 @@
     <gazebo reference="left_wheel">
         <material>Gazebo/Black</material>
+        <mu1 value="0.8"/>
+        <mu2 value="0.8"/>
     </gazebo>
     <joint name="caster_wheel_joint" type="fixed">
@@ -202,5 +222,5 @@
                 </ros>
                 <output_type>sensor_msgs/Range</output_type>
-                <!-- <frame_name> ommited, will default to range_link -->
+                <frame_name>laser_link</frame_name>
             </plugin>
         </sensor>

Commit message: Add gripper in simulation, breaks real robot

File: src/mek_lilrobot/description/robot_core.xacro (robot description, xacro)
@@ -16,20 +16,19 @@
         <parent link="base_link" />
         <child link="chassis" />
-        <origin xyz="-0.042025 0 0.032925" />
+        <origin xyz="0 0 0" />
     </joint>
     <link name="chassis">
         <visual>
             <geometry>
-                <box size="0.1222 0.10825 0.005" />
-            </geometry>
-            <material name="white" />
-        </visual>
-        <collision>
-            <geometry>
-                <box size="0.1222 0.10825 0.005" />
-            </geometry>
-        </collision>
-        <xacro:inertial_box mass="0.5" x="0.1222" y="0.10825" z="0.005">
-            <origin xyz="0 0 0" rpy="0 0 0" />
+                <mesh filename="$(find mek_lilrobot)/description/mek_chassis.stl"/>
+            </geometry>
+        </visual>
+        <collision>
+            <geometry>
+                <mesh filename="$(find mek_lilrobot)/description/mek_chassis_collision.stl"/>
+            </geometry>
+        </collision>
+        <xacro:inertial_box mass="0.8" x="0.1222" y="0.10825" z="0.005">
+            <origin xyz="-0.042 0 0.027" rpy="0 0 0" />
         </xacro:inertial_box>
     </link>
@@ -226,3 +225,56 @@
         </sensor>
     </gazebo>
+    <!-- Gripper -->
+    <link name="gripper_right_link">
+        <visual>
+            <geometry>
+                <mesh filename="$(find mek_lilrobot)/description/gripper_right_visual.stl"/>
+            </geometry>
+            <material name="white"/>
+        </visual>
+        <collision>
+            <geometry>
+                <mesh filename="$(find mek_lilrobot)/description/gripper_right_collision.stl"/>
+            </geometry>
+        </collision>
+        <xacro:inertial_box mass="0.05" x="0.04" y="0.005" z="0.03">
+            <origin xyz="0.020 0 -0.015" rpy="0 0 0"/>
+        </xacro:inertial_box>
+    </link>
+    <joint type="revolute" name="gripper_right_joint">
+        <parent link="base_link"/>
+        <child link="gripper_right_link"/>
+        <origin xyz="0.0021 -0.010 0.03175" rpy="0 0 0"/>
+        <axis xyz="0 0 1"/>
+        <limit effort="1" velocity="1" lower="-0.74" upper="0.219"/>
+    </joint>
+    <link name="gripper_left_link">
+        <visual>
+            <geometry>
+                <mesh filename="$(find mek_lilrobot)/description/gripper_left_visual.stl"/>
+            </geometry>
+            <material name="white"/>
+        </visual>
+        <collision>
+            <geometry>
+                <mesh filename="$(find mek_lilrobot)/description/gripper_left_collision.stl"/>
+            </geometry>
+        </collision>
+        <xacro:inertial_box mass="0.05" x="0.04" y="0.005" z="0.03">
+            <origin xyz="0.020 0 0.015" rpy="0 0 0"/>
+        </xacro:inertial_box>
+    </link>
+    <joint type="revolute" name="gripper_left_joint">
+        <parent link="base_link"/>
+        <child link="gripper_left_link"/>
+        <origin xyz="0.0021 0.010 0.03175" rpy="${pi} 0 0"/>
+        <axis xyz="0 0 -1"/>
+        <limit effort="1" velocity="1" lower="-0.219" upper="0.74"/>
+    </joint>
+    <gazebo reference="gripper_right_link">
+        <self_collide>1</self_collide>
+    </gazebo>
+    <gazebo reference="gripper_left_link">
+        <self_collide>1</self_collide>
+    </gazebo>
 </robot>

File: src/mek_lilrobot/description/ros2_control.xacro (robot description, xacro)
@@ -39,5 +39,5 @@
                 <command_interface name="velocity">
                     <param name="min">-1</param>
-                    <param name="min">1</param>
+                    <param name="max">1</param>
                 </command_interface>
                 <state_interface name="velocity"/>
@@ -47,8 +47,19 @@
                 <command_interface name="velocity">
                     <param name="min">-1</param>
-                    <param name="min">1</param>
+                    <param name="max">1</param>
                 </command_interface>
                 <state_interface name="velocity"/>
                 <state_interface name="position"/>
+            </joint>
+            <joint name="gripper_right_joint">
+                <command_interface name="effort">
+                    <param name="min">-0.1</param>
+                    <param name="max">0.1</param>
+                </command_interface>
+            </joint>
+            <joint name="gripper_left_joint">
+                <param name="mimic">gripper_right_joint</param>
+                <param name="multiplier">-1</param>
+                <command_interface name="effort"/>
             </joint>
         </ros2_control>
