Commit message: Real robot working with ros2_control, gazebo broken

File: src/mek_lilrobot/description/ros2_control.xacro (robot description, xacro)
@@ -1,4 +1,33 @@
 <?xml version="1.0"?>
 <robot xmlns:xacro="http://www.ros.org/wiki/xacro">
+    <ros2_control name="RealRobot" type="system">
+        <hardware>
+            <plugin>diffdrive_arduino/DiffDriveArduino</plugin>
+            <param name="left_wheel_name">left_wheel_joint</param>
+            <param name="right_wheel_name">right_wheel_joint</param>
+            <param name="loop_rate">30</param>
+            <param name="device">/dev/ttyACM0</param>
+            <param name="baud_rate">57600</param>
+            <param name="timeout">1000</param>
+            <param name="enc_counts_per_rev">8340</param>
+        </hardware>
+        <joint name="left_wheel_joint">
+            <command_interface name="velocity">
+                <param name="min">-1</param>
+                <param name="min">1</param>
+            </command_interface>
+            <state_interface name="velocity"/>
+            <state_interface name="position"/>
+        </joint>
+        <joint name="right_wheel_joint">
+            <command_interface name="velocity">
+                <param name="min">-1</param>
+                <param name="min">1</param>
+            </command_interface>
+            <state_interface name="velocity"/>
+            <state_interface name="position"/>
+        </joint>
+    </ros2_control>
+    	<!-- Gazebo
     <ros2_control name="GazeboSystem" type="system">
         <hardware>
@@ -27,3 +56,4 @@
         </plugin>
     </gazebo>
+        -->
 </robot>

Commit message: Integration, everything works on real robot!

File: src/mek_lilrobot/description/ros2_control.xacro (robot description, xacro)
@@ -28,4 +28,10 @@
                 <state_interface name="velocity"/>
                 <state_interface name="position"/>
+            </joint>
+            <joint name="gripper_right_joint">
+                <command_interface name="effort">
+                    <param name="min">-0.1</param>
+                    <param name="max">0.1</param>
+                </command_interface>
             </joint>
         </ros2_control>
@@ -66,5 +72,5 @@
         <gazebo>
             <plugin name="gazebo_ros2_control" filename="libgazebo_ros2_control.so">
-                <parameters>$(find mek_lilrobot)/config/controllers.yaml</parameters>
+                <parameters>$(find mek_lilrobot)/config/sim_controllers.yaml</parameters>
             </plugin>
         </gazebo>
